File: pcb/switch42.kicad_pcb (KiCad board)
At the start: 2 copper layers, 91 x 55 mm, 35 parts, among them J1 Conn_01x02, J2 MJ-4PP-9, J3 MJ-4PP-9, Q1 Q_NPN_ECB, SW1 SW_PUSH, SW2 SW_PUSH, SW4 SW_PUSH, SW5 SW_PUSH, SW7 SW_PUSH, U1 ProMicro

Commit message: Change register and capacitor values
Other:
- board text added: "1uF"
- board text added: "47K"
- board text removed: "10K"
- board text removed: "10uF"
Changed lines of the file:
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@@
     (effects (font (size 0.7 0.7) (thickness 0.15)) (justify mirror))
   )
-  (gr_text 10K (at 103.5 78.25 180) (layer B.SilkS)
+  (gr_text 47K (at 103.5 78.25 180) (layer B.SilkS)
     (effects (font (size 0.7 0.7) (thickness 0.15)) (justify mirror))
   )
-  (gr_text 10K (at 107.5 78.25 180) (layer B.SilkS)
+  (gr_text 47K (at 107.5 78.25 180) (layer B.SilkS)
     (effects (font (size 0.7 0.7) (thickness 0.15)) (justify mirror))
   )
@@
     (effects (font (size 0.7 0.7) (thickness 0.15)) (justify mirror))
   )
-  (gr_text 10uF (at 117.25 69.5 180) (layer B.SilkS)
+  (gr_text 1uF (at 117.25 69.5 180) (layer B.SilkS)
     (effects (font (size 0.7 0.7) (thickness 0.15)) (justify mirror))
   )
